File: kicad/sata_psu.kicad_sch (KiCad schematic)
At the start: 0 parts

Commit message: v2: per-port 5V buck with 0R neighbour sharing, plus rail indicators
Every port now has its own local 5V node and its own buck footprint, with
adjacent nodes joined by 0R links (R61-R64). How a port gets its 5V is a
populate choice rather than a layout one -- BUCKS/LINKS at the top of
gen_sch.py is the whole configuration, and the lands are always present.

This closes v1's largest open issue. One 3A TPS563200 was under-rated
against a five-bay 5V rail; capping a buck at a three-port group makes its
worst case 2.1A and the same part is correctly sized.

Indicators: one 12V LED on the common rail, tapped after Q8 so it also
proves the reverse-polarity guard conducts, and one 5V LED per port on the
local node at the header, so it lights whether that port's 5V came from its
own buck or across a link.

verify.py gains check 5, the rail populate rules. A DNP part is still a
wire in the netlist, so a build that fits R63 with both U2 and U4 populated
passes ERC and netlist equivalence and parallels two regulators on the
bench. Nothing else can catch it. It also refuses groups over three ports
and any link carrying more than one port's current.

Also fixed: check_layout.py reported "0 symbols checked" and PASSED after
KiCad re-saved the sheets in its own format, because text[text.find(m):]
yields the last character rather than "" when the marker is absent, so the
`or text` fallback never fired. It now fails loudly when it parses nothing.

Schematic verified (ERC clean, 50 nets equivalent to the independent SKiDL
description, pins match pads). Board placed at 64.9 x 76.0 mm, 112 parts,
0 DRC violations. Routing still not started.

Co-Authored-By: Claude Opus 5 <noreply@anthropic.com>
Other:
- removed sheet 5V buck regulator
- added sheet 5V rail links (sata_psu_rails.kicad_sch)
- note added: "5V rails: U2 -> ports 1,2,3 | U4 -> ports 4,5"
- note added: "Single 12V brick, five analog-staggered channels, per-port 5V buck"
- note removed: "Single 12V brick, onboard 5V buck, five analog-staggered channels"
Changed lines of the file:
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@@
     (effects (font (size 3.5 3.5)) (justify left bottom))
   )
-  (text "Single 12V brick, onboard 5V buck, five analog-staggered channels"
+  (text "Single 12V brick, five analog-staggered channels, per-port 5V buck"
     (exclude_from_sim no)
     (at 38.1 31.75 0)
     (effects (font (size 2.0 2.0)) (justify left bottom))
+  )
+  (text "5V rails: U2 -> ports 1,2,3 | U4 -> ports 4,5"
+    (exclude_from_sim no)
+    (at 38.1 36.83 0)
+    (effects (font (size 1.8 1.8)) (justify left bottom))
   )
   (sheet
@@
     (stroke (width 0.1524) (type solid))
     (fill (color 0 0 0 0.0000))
-    (property "Sheetname" "5V buck regulator" (at 25.4 88.2 0) (effects (font (size 1.524 1.524)) (justify left bottom)))
-    (property "Sheetfile" "sata_psu_buck.kicad_sch" (at 25.4 115.70000000000002 0) (effects (font (size 1.524 1.524)) (justify left top)))
+    (property "Sheetname" "5V rail links" (at 25.4 88.2 0) (effects (font (size 1.524 1.524)) (justify left bottom)))
+    (property "Sheetfile" "sata_psu_rails.kicad_sch" (at 25.4 115.70000000000002 0) (effects (font (size 1.524 1.524)) (justify left top)))
     (instances
       (project "sata_psu"
