File: kicad/sata_psu_channel1.kicad_sch (KiCad schematic)
At the start: 8 parts, among them J1 12V/GND/GND/5V, Q1 AO3401A

Commit message: v2: per-port 5V buck with 0R neighbour sharing, plus rail indicators
Every port now has its own local 5V node and its own buck footprint, with
adjacent nodes joined by 0R links (R61-R64). How a port gets its 5V is a
populate choice rather than a layout one -- BUCKS/LINKS at the top of
gen_sch.py is the whole configuration, and the lands are always present.

This closes v1's largest open issue. One 3A TPS563200 was under-rated
against a five-bay 5V rail; capping a buck at a three-port group makes its
worst case 2.1A and the same part is correctly sized.

Indicators: one 12V LED on the common rail, tapped after Q8 so it also
proves the reverse-polarity guard conducts, and one 5V LED per port on the
local node at the header, so it lights whether that port's 5V came from its
own buck or across a link.

verify.py gains check 5, the rail populate rules. A DNP part is still a
wire in the netlist, so a build that fits R63 with both U2 and U4 populated
passes ERC and netlist equivalence and parallels two regulators on the
bench. Nothing else can catch it. It also refuses groups over three ports
and any link carrying more than one port's current.

Also fixed: check_layout.py reported "0 symbols checked" and PASSED after
KiCad re-saved the sheets in its own format, because text[text.find(m):]
yields the last character rather than "" when the marker is absent, so the
`or text` fallback never fired. It now fails loudly when it parses nothing.

Schematic verified (ERC clean, 50 nets equivalent to the independent SKiDL
description, pins match pads). Board placed at 64.9 x 76.0 mm, 112 parts,
0 DRC violations. Routing still not started.

Co-Authored-By: Claude Opus 5 <noreply@anthropic.com>
Parts:
- removed D1: 8.2V, Diode_SMD:D_SOD-123, symbol Device:D_Zener
- removed R1: 220k, Resistor_SMD:R_0603_1608Metric, symbol Device:R
- added C14: 10uF/50V, Capacitor_SMD:C_1206_3216Metric, symbol Device:C
- added C15, C16: 100nF, Capacitor_SMD:C_0603_1608Metric, symbol Device:C
- added C17, C18: 22uF/25V, Capacitor_SMD:C_1206_3216Metric, symbol Device:C
- added D11: 8.2V, Diode_SMD:D_SOD-123, symbol Device:D_Zener
- added D12: GRN, LED_SMD:LED_0603_1608Metric, symbol Device:LED
- added L1: 4.7uH/4.5A, Inductor_SMD:L_Bourns_SRN6045TA, symbol Device:L
- added R11: 220k, Resistor_SMD:R_0603_1608Metric, symbol Device:R
- added R12: 56k, Resistor_SMD:R_0603_1608Metric, symbol Device:R
- added R13: 10k, Resistor_SMD:R_0603_1608Metric, symbol Device:R
- added R14: 100k, Resistor_SMD:R_0603_1608Metric, symbol Device:R
- added R15: 1.5k, Resistor_SMD:R_0603_1608Metric, symbol Device:R
- added U1: TPS563200, Package_TO_SOT_SMD:SOT-23-6, symbol Regulator_Switching:TPS563200
Connections:
- net 12V_MAIN: now also C14.1, C15.1, D11.1 (K), R14.1, U1.3 (VIN)
- net GND: now also C14.2, C15.2, C17.2, C18.2, R11.2, R13.2, R15.2, U1.1 (GND)
- net at C11.2, Q1.1 (G): now also D11.2 (A), R11.1
- net 5V_MAIN renamed 5V_1
- net 5V_1: now also C17.1, C18.1, D12.2 (A), L1.2, R12.1
- new net: D12.1 (K), R15.1
- new net: R14.2, U1.5 (EN)
- new net: R12.2, R13.1, U1.4 (VFB)
- new net: C16.1, L1.1, U1.2 (SW)
- new net: C16.2, U1.6 (VBST)
Other:
- note added: "(5 - 2.0) / 1.5k = 2.0mA"
- note added: "C11=1uF with R11=220k sets turn-on at ~0.2s"
- note added: "Channel 1 - staggered high-side switch + local 5V"
- note added: "D11 clamps Vgs to 8.2V; AO3401A is rated +/-12V"
- note added: "Max load is a 3-port group; see BUCKS/LINKS in gen_sch.py"
- note added: "Port 1 local 5V buck [DNP - this port takes 5V from a neighbour]"
- note added: "Vout = 0.768V x (1 + R12/R13) = 0.768 x (1 + 56k/10k) = 5.07V"
- note removed: "C11=1uF with R1=220k sets turn-on at ~0.2s"
- note removed: "Channel 1 - staggered high-side switch"
- note removed: "D1 clamps Vgs to 8.2V; AO3401A is rated +/-12V"
