File: kicad/sata_psu_channel4.kicad_sch (KiCad schematic)
At the start: 8 parts, among them J4 12V/GND/GND/5V, Q4 AO3401A

Commit message: v2: per-port 5V buck with 0R neighbour sharing, plus rail indicators
Every port now has its own local 5V node and its own buck footprint, with
adjacent nodes joined by 0R links (R61-R64). How a port gets its 5V is a
populate choice rather than a layout one -- BUCKS/LINKS at the top of
gen_sch.py is the whole configuration, and the lands are always present.

This closes v1's largest open issue. One 3A TPS563200 was under-rated
against a five-bay 5V rail; capping a buck at a three-port group makes its
worst case 2.1A and the same part is correctly sized.

Indicators: one 12V LED on the common rail, tapped after Q8 so it also
proves the reverse-polarity guard conducts, and one 5V LED per port on the
local node at the header, so it lights whether that port's 5V came from its
own buck or across a link.

verify.py gains check 5, the rail populate rules. A DNP part is still a
wire in the netlist, so a build that fits R63 with both U2 and U4 populated
passes ERC and netlist equivalence and parallels two regulators on the
bench. Nothing else can catch it. It also refuses groups over three ports
and any link carrying more than one port's current.

Also fixed: check_layout.py reported "0 symbols checked" and PASSED after
KiCad re-saved the sheets in its own format, because text[text.find(m):]
yields the last character rather than "" when the marker is absent, so the
`or text` fallback never fired. It now fails loudly when it parses nothing.

Schematic verified (ERC clean, 50 nets equivalent to the independent SKiDL
description, pins match pads). Board placed at 64.9 x 76.0 mm, 112 parts,
0 DRC violations. Routing still not started.

Co-Authored-By: Claude Opus 5 <noreply@anthropic.com>
Parts:
- removed D4: 8.2V, Diode_SMD:D_SOD-123, symbol Device:D_Zener
- removed R4: 220k, Resistor_SMD:R_0603_1608Metric, symbol Device:R
- added C44: 10uF/50V, Capacitor_SMD:C_1206_3216Metric, symbol Device:C
- added C45, C46: 100nF, Capacitor_SMD:C_0603_1608Metric, symbol Device:C
- added C47, C48: 22uF/25V, Capacitor_SMD:C_1206_3216Metric, symbol Device:C
- added D41: 8.2V, Diode_SMD:D_SOD-123, symbol Device:D_Zener
- added D42: GRN, LED_SMD:LED_0603_1608Metric, symbol Device:LED
- added L4: 4.7uH/4.5A, Inductor_SMD:L_Bourns_SRN6045TA, symbol Device:L
- added R41: 220k, Resistor_SMD:R_0603_1608Metric, symbol Device:R
- added R42: 56k, Resistor_SMD:R_0603_1608Metric, symbol Device:R
- added R43: 10k, Resistor_SMD:R_0603_1608Metric, symbol Device:R
- added R44: 100k, Resistor_SMD:R_0603_1608Metric, symbol Device:R
- added R45: 1.5k, Resistor_SMD:R_0603_1608Metric, symbol Device:R
- added U4: TPS563200, Package_TO_SOT_SMD:SOT-23-6, symbol Regulator_Switching:TPS563200
Connections:
- net 12V_MAIN: now also C44.1, C45.1, D41.1 (K), R44.1, U4.3 (VIN)
- net GND: now also C44.2, C45.2, C47.2, C48.2, R41.2, R43.2, R45.2, U4.1 (GND)
- net at C41.2, Q4.1 (G): now also D41.2 (A), R41.1
- net 5V_MAIN renamed 5V_4
- net 5V_4: now also C47.1, C48.1, D42.2 (A), L4.2, R42.1
- new net: C46.1, L4.1, U4.2 (SW)
- new net: R42.2, R43.1, U4.4 (VFB)
- new net: R44.2, U4.5 (EN)
- new net: C46.2, U4.6 (VBST)
- new net: D42.1 (K), R45.1
Other:
- note added: "(5 - 2.0) / 1.5k = 2.0mA"
- note added: "C41=10uF with R41=220k sets turn-on at ~2.2s"
- note added: "Channel 4 - staggered high-side switch + local 5V"
- note added: "D41 clamps Vgs to 8.2V; AO3401A is rated +/-12V"
- note added: "Max load is a 3-port group; see BUCKS/LINKS in gen_sch.py"
- note added: "Port 4 local 5V buck"
- note added: "Vout = 0.768V x (1 + R42/R43) = 0.768 x (1 + 56k/10k) = 5.07V"
- note removed: "C41=10uF with R4=220k sets turn-on at ~2.2s"
- note removed: "Channel 4 - staggered high-side switch"
- note removed: "D4 clamps Vgs to 8.2V; AO3401A is rated +/-12V"
