File: kicad/sata_psu_channel5.kicad_sch (KiCad schematic)
At the start: 8 parts, among them J5 12V/GND/GND/5V, Q5 AO3401A

Commit message: v2: per-port 5V buck with 0R neighbour sharing, plus rail indicators
Every port now has its own local 5V node and its own buck footprint, with
adjacent nodes joined by 0R links (R61-R64). How a port gets its 5V is a
populate choice rather than a layout one -- BUCKS/LINKS at the top of
gen_sch.py is the whole configuration, and the lands are always present.

This closes v1's largest open issue. One 3A TPS563200 was under-rated
against a five-bay 5V rail; capping a buck at a three-port group makes its
worst case 2.1A and the same part is correctly sized.

Indicators: one 12V LED on the common rail, tapped after Q8 so it also
proves the reverse-polarity guard conducts, and one 5V LED per port on the
local node at the header, so it lights whether that port's 5V came from its
own buck or across a link.

verify.py gains check 5, the rail populate rules. A DNP part is still a
wire in the netlist, so a build that fits R63 with both U2 and U4 populated
passes ERC and netlist equivalence and parallels two regulators on the
bench. Nothing else can catch it. It also refuses groups over three ports
and any link carrying more than one port's current.

Also fixed: check_layout.py reported "0 symbols checked" and PASSED after
KiCad re-saved the sheets in its own format, because text[text.find(m):]
yields the last character rather than "" when the marker is absent, so the
`or text` fallback never fired. It now fails loudly when it parses nothing.

Schematic verified (ERC clean, 50 nets equivalent to the independent SKiDL
description, pins match pads). Board placed at 64.9 x 76.0 mm, 112 parts,
0 DRC violations. Routing still not started.

Co-Authored-By: Claude Opus 5 <noreply@anthropic.com>
Parts:
- removed D5: 8.2V, Diode_SMD:D_SOD-123, symbol Device:D_Zener
- removed R5: 220k, Resistor_SMD:R_0603_1608Metric, symbol Device:R
- added C54: 10uF/50V, Capacitor_SMD:C_1206_3216Metric, symbol Device:C
- added C55, C56: 100nF, Capacitor_SMD:C_0603_1608Metric, symbol Device:C
- added C57, C58: 22uF/25V, Capacitor_SMD:C_1206_3216Metric, symbol Device:C
- added D51: 8.2V, Diode_SMD:D_SOD-123, symbol Device:D_Zener
- added D52: GRN, LED_SMD:LED_0603_1608Metric, symbol Device:LED
- added L5: 4.7uH/4.5A, Inductor_SMD:L_Bourns_SRN6045TA, symbol Device:L
- added R51: 220k, Resistor_SMD:R_0603_1608Metric, symbol Device:R
- added R52: 56k, Resistor_SMD:R_0603_1608Metric, symbol Device:R
- added R53: 10k, Resistor_SMD:R_0603_1608Metric, symbol Device:R
- added R54: 100k, Resistor_SMD:R_0603_1608Metric, symbol Device:R
- added R55: 1.5k, Resistor_SMD:R_0603_1608Metric, symbol Device:R
- added U5: TPS563200, Package_TO_SOT_SMD:SOT-23-6, symbol Regulator_Switching:TPS563200
Connections:
- net 12V_MAIN: now also C54.1, C55.1, D51.1 (K), R54.1, U5.3 (VIN)
- net GND: now also C54.2, C55.2, C57.2, C58.2, R51.2, R53.2, R55.2, U5.1 (GND)
- net at C51.2, Q5.1 (G): now also D51.2 (A), R51.1
- net 5V_MAIN renamed 5V_5
- net 5V_5: now also C57.1, C58.1, D52.2 (A), L5.2, R52.1
- new net: C56.1, L5.1, U5.2 (SW)
- new net: R52.2, R53.1, U5.4 (VFB)
- new net: R54.2, U5.5 (EN)
- new net: C56.2, U5.6 (VBST)
- new net: D52.1 (K), R55.1
Other:
- note added: "(5 - 2.0) / 1.5k = 2.0mA"
- note added: "C51=22uF with R51=220k sets turn-on at ~4.8s"
- note added: "Channel 5 - staggered high-side switch + local 5V"
- note added: "D51 clamps Vgs to 8.2V; AO3401A is rated +/-12V"
- note added: "Max load is a 3-port group; see BUCKS/LINKS in gen_sch.py"
- note added: "Port 5 local 5V buck [DNP - this port takes 5V from a neighbour]"
- note added: "Vout = 0.768V x (1 + R52/R53) = 0.768 x (1 + 56k/10k) = 5.07V"
- note removed: "C51=22uF with R5=220k sets turn-on at ~4.8s"
- note removed: "Channel 5 - staggered high-side switch"
- note removed: "D5 clamps Vgs to 8.2V; AO3401A is rated +/-12V"
